File: petfeeder/Keyboard_LCD.sch (KiCad schematic (older format))
At the start: 18 parts, among them J1 External UART Conn., J2 Ext. Motor Conn., J3 Ext. Servo Conn., J4 Ext. LCD Conn., J5 Ext. Keyboard Conn., J6 Ext. Balance Conn., Q1 BC237, U1 ESP-12F, U3 DS1307+, U4 L7812, U5 L7805, Y1 32kHz

Commit message: Atualizações
Parts:
- removed C3: C, symbol Device:C
- removed J1: External UART Conn., symbol Connector:Conn_01x03_Female
- removed J2: Ext. Motor Conn., symbol Connector:Conn_01x02_Male
- removed J3: Ext. Servo Conn., symbol Connector:Conn_01x03_Female
- removed J4: Ext. LCD Conn., symbol Connector:Conn_01x04_Female
- removed J5: Ext. Keyboard Conn., symbol Connector:Conn_01x08_Male
- removed J6: Ext. Balance Conn., symbol Connector:Conn_01x03_Male
- removed Q1: BC237, Package_TO_SOT_THT:TO-92_Inline, symbol Transistor_BJT:BC237
- removed R1, R5: 10kR, symbol Device:R
- removed R2: R, symbol Device:R
- removed R3, R4: 1kR, symbol Device:R
- removed U1: ESP-12F, RF_Module:ESP-12E, symbol RF_Module:ESP-12F
- removed U3: DS1307+, Package_DIP:DIP-8_W7.62mm, symbol Timer_RTC:DS1307+
- removed U4: L7812, symbol Regulator_Linear:L7812
- removed U5: L7805, symbol Regulator_Linear:L7805
- removed Y1: 32kHz, symbol Device:Crystal
- added C1: 150uF, symbol Device:C
- added C2: 10pF, symbol Device:C
- added R6: 2.2kR, symbol Device:R
- added R7: 200R, symbol Device:R
- added U2: 4022, symbol 4xxx:4022
- added U6: NE555P, Package_DIP:DIP-8_W7.62mm, symbol Timer:NE555P
- added U?: PIC16F84A-XXP, symbol MCU_Microchip_PIC16:PIC16F84A-XXP
Connections:
- net +5V: now also C2.1, R7.2, U2.16 (VDD), U6.4 (R), U6.8 (VCC)
- net GND: now also C1.1, C2.2, U2.13 (CKEN), U2.15 (Reset), U2.8 (VSS), U6.1 (GND)
- net column1: now also U2.2 (Q0)
- net column2: now also U2.1 (Q1)
- net column3: now also U2.3 (Q2)
- net column4: now also U2.7 (Q3)
- new net: C1.2, R6.1, U6.2 (TR), U6.6 (THR)
- new net: R6.2, R7.1, U6.7 (DIS)
- new net CLK: U2.14 (CLK), U6.3 (Q)
- no-connect marks 7 -> 6
Other:
- note added: "Keyboard's columns pulser\n"
- note removed: "Engines Circuits"
- note removed: "External LCD and Keyboard Circuits"
- note removed: "Main Circuit\n\n"
