File: Electronic Schematic/Battery Schema.sch (KiCad schematic (older format))
At the start: 18 parts, among them J1 External UART Conn., J2 Ext. Motor Conn., J3 Ext. Servo Conn., J4 Ext. LCD Conn., J5 Ext. Keyboard Conn., J6 Ext. Balance Conn., Q1 BC237, U1 ESP-12F, U3 DS1307+, U4 L7812, U5 L7805, Y1 32kHz

Commit message: Hadware 100%
Parts:
- removed C3: C, symbol Device:C
- removed J1: External UART Conn., symbol Connector:Conn_01x03_Female
- removed J2: Ext. Motor Conn., symbol Connector:Conn_01x02_Male
- removed J3: Ext. Servo Conn., symbol Connector:Conn_01x03_Female
- removed J4: Ext. LCD Conn., symbol Connector:Conn_01x04_Female
- removed J5: Ext. Keyboard Conn., symbol Connector:Conn_01x08_Male
- removed J6: Ext. Balance Conn., symbol Connector:Conn_01x03_Male
- removed Q1: BC237, Package_TO_SOT_THT:TO-92_Inline, symbol Transistor_BJT:BC237
- removed R1, R5: 10kR, symbol Device:R
- removed R2: R, symbol Device:R
- removed R3, R4: 1kR, symbol Device:R
- removed U1: ESP-12F, RF_Module:ESP-12E, symbol RF_Module:ESP-12F
- removed U3: DS1307+, Package_DIP:DIP-8_W7.62mm, symbol Timer_RTC:DS1307+
- removed U4: L7812, symbol Regulator_Linear:L7812
- removed U5: L7805, symbol Regulator_Linear:L7805
- removed Y1: 32kHz, symbol Device:Crystal
- added C8: C, symbol Device:C
- added C9: 300pF, symbol Device:C
- added D3, D4: 1N4001, Diode_THT:D_DO-41_SOD81_P10.16mm_Horizontal, symbol Diode:1N4001
- added F1: Fuse, symbol Device:Fuse
- added J4: Ext. Battery Conn., symbol Connector:Conn_01x02_Female
- added R10, R9: 100kR, symbol Device:R
- added R8: R, symbol Device:R
- added U8: LTC4055, Package_DFN_QFN:QFN-16-1EP_4x4mm_P0.65mm_EP2.15x2.15mm, symbol Battery_Management:LTC4055
Connections:
- net labels added: +3.3V_OUT, +5V_BAT, +5V_OUT
- net labels removed: +12V, RX, SCL, SDA, TX, balança, column1, column2, column3, column4, flash, line1, line2, line3, line4, motor, motor+, motor-, servo, servo+, servo-
- wire segments 79 -> 37
- no-connect marks 7 -> 4
Other:
- note added: "Battery Charging and Backup Circuit"
- note removed: "Engines Circuits"
- note removed: "External LCD and Keyboard Circuits"
- note removed: "Main Circuit\n\n"
